Commit message: fixed base size and increased the size

File: parking_barrier_description/urdf/parking_barrier.xacro (robot description, xacro)
@@ -6,7 +6,7 @@
 <link name="base_link">
   <inertial>
-    <origin xyz="-0.0056187645592535584 -0.04116590365886497 0.47494061878933524" rpy="0 0 0"/>
-    <mass value="21.5338040215956"/>
-    <inertia ixx="2.234201" iyy="2.452824" izz="0.81716" ixy="-0.019409" iyz="0.017759" ixz="0.10187"/>
+    <origin xyz="0.08849577120552374 -0.04294425760323125 0.4483427058249352" rpy="0 0 0"/>
+    <mass value="22.844754021591662"/>
+    <inertia ixx="2.588206" iyy="6.739632" izz="4.927033" ixy="-0.042188" iyz="9e-06" ixz="1.041216"/>
   </inertial>
   <visual>

Commit message: Fixed the position controller

File: parking_barrier_description/urdf/parking_barrier.xacro (robot description, xacro)
@@ -51,3 +51,12 @@
   <limit upper="0.0" lower="-1.570796" effort="100" velocity="100"/>
 </joint>
+    <transmission name="Rev1_trans" type="SimpleTransmission">
+			<type>transmission_interface/SimpleTransmission</type>
+			<actuator name="Rev1_motor">
+				<mechanicalReduction>1</mechanicalReduction>
+			</actuator>
+			<joint name="Rev1">
+				<hardwareInterface>hardware_interface/PositionJointInterface</hardwareInterface>
+			</joint>
+		</transmission>
 </robot>

Commit message: added parking sim

File: parking_barrier_description/urdf/parking_barrier.xacro (robot description, xacro)
@@ -7,5 +7,5 @@
   <inertial>
     <origin xyz="0.08849577120552374 -0.04294425760323125 0.4483427058249352" rpy="0 0 0"/>
-    <mass value="22.844754021591662"/>
+    <mass value="2220.844754021591662"/>
     <inertia ixx="2.588206" iyy="6.739632" izz="4.927033" ixy="-0.042188" iyz="9e-06" ixz="1.041216"/>
   </inertial>

Commit message: Updates env_hooks, adds launch files

File: parking_barrier_description/urdf/parking_barrier.xacro (robot description, xacro)
@@ -13,5 +13,5 @@
     <origin xyz="0 0 0" rpy="0 0 0"/>
     <geometry>
-      <mesh filename="package://parking_barrier_description/meshes/base_link.stl" scale="0.001 0.001 0.001"/>
+      <mesh filename="package://parking_sim/models/barrier/meshes/barrier0.dae" scale="1 1 1"/>
     </geometry>
     <material name="silver"/>
@@ -20,5 +20,5 @@
     <origin xyz="0 0 0" rpy="0 0 0"/>
     <geometry>
-      <mesh filename="package://parking_barrier_description/meshes/base_link.stl" scale="0.001 0.001 0.001"/>
+      <mesh filename="package://parking_sim/models/barrier/meshes/barrier0.dae" scale="1 1 1"/>
     </geometry>
   </collision>
@@ -33,5 +33,5 @@
     <origin xyz="0.016028 -0.106468 -0.828993" rpy="0 0 0"/>
     <geometry>
-      <mesh filename="package://parking_barrier_description/meshes/barrier_1.stl" scale="0.001 0.001 0.001"/>
+      <mesh filename="package://parking_sim/models/barrier/meshes/barrier1.dae" scale="1 1 1"/>
     </geometry>
     <material name="silver"/>
@@ -40,5 +40,5 @@
     <origin xyz="0.016028 -0.106468 -0.828993" rpy="0 0 0"/>
     <geometry>
-      <mesh filename="package://parking_barrier_description/meshes/barrier_1.stl" scale="0.001 0.001 0.001"/>
+      <mesh filename="package://parking_sim/models/barrier/meshes/barrier1.dae" scale="1 1 1"/>
     </geometry>
   </collision>
@@ -51,12 +51,3 @@
   <limit upper="0.0" lower="-1.570796" effort="100" velocity="100"/>
 </joint>
-    <transmission name="Rev1_trans" type="SimpleTransmission">
-			<type>transmission_interface/SimpleTransmission</type>
-			<actuator name="Rev1_motor">
-				<mechanicalReduction>1</mechanicalReduction>
-			</actuator>
-			<joint name="Rev1">
-				<hardwareInterface>hardware_interface/PositionJointInterface</hardwareInterface>
-			</joint>
-		</transmission>
 </robot>
